File: TESTER_BTR_12.sch (KiCad schematic (older format))
At the start: 8 parts, among them J5 Conn_01x01_Female, J6 Conn_01x01_Female, J7 Conn_01x01_Female, J8 Conn_01x01_Female, Q1 Conn_01x01_Female

Commit message: Added the .txt file and edited the line names
Connections:
- net Q1: now reaches J5.1 (Pin_1), Q1.1 (Pin_1)
- net VIN: now reaches J6.1 (Pin_1), VIN1.1 (Pin_1)
- net GND: now reaches GND1.1 (Pin_1), J7.1 (Pin_1)
- net VOUT: now reaches J8.1 (Pin_1), VOUT1.1 (Pin_1)
Changed lines of the file:
@@
 $EndComp
-Wire Wire Line
-	5000 2350 6000 2350
 Wire Wire Line
 	5000 2600 6000 2600
@@
 Wire Wire Line
 	5000 3100 6000 3100
+Wire Wire Line
+	5000 2350 6000 2350
+Text Label 5550 2350 0    50   ~ 0
+VOUT
+Text Label 5550 2600 0    50   ~ 0
+GND
+Text Label 5550 2850 0    50   ~ 0
+VIN
+Text Label 5550 3100 0    50   ~ 0
+Q1
 $EndSCHEMATC
